File: electronics/board/hardware.kicad_sch (KiCad schematic)
At the start: 1 part, among them J1 0513386473

Commit message: Working on the routing.
Changed lines of the file:
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@@
     (effects (font (size 1.27 1.27)) (justify left bottom))
   )
-  (label "ODT" (at 73.025 60.96 0)
+  (label "ODT_0" (at 73.025 60.96 0)
     (effects (font (size 1.27 1.27)) (justify left bottom))
   )
@@
     (effects (font (size 1.27 1.27)) (justify right bottom))
   )
-  (label "CKE" (at 219.075 42.545 180)
+  (label "CKE_1" (at 219.075 42.545 180)
     (effects (font (size 1.27 1.27)) (justify right bottom))
   )
@@
     (effects (font (size 1.27 1.27)) (justify right bottom))
   )
-  (label "CKE" (at 73.025 118.11 0)
+  (label "CKE_0" (at 73.025 118.11 0)
     (effects (font (size 1.27 1.27)) (justify left bottom))
   )
@@
     (effects (font (size 1.27 1.27)) (justify right bottom))
   )
-  (label "DQS" (at 73.025 149.225 0)
+  (label "UDQS" (at 73.025 149.225 0)
     (effects (font (size 1.27 1.27)) (justify left bottom))
   )
@@
     (effects (font (size 1.27 1.27)) (justify right bottom))
   )
-  (label "~{CS}" (at 219.075 51.435 180)
+  (label "~{CS_1}" (at 219.075 51.435 180)
     (effects (font (size 1.27 1.27)) (justify right bottom))
   )
@@
     (effects (font (size 1.27 1.27)) (justify left bottom))
   )
-  (label "CKE" (at 73.025 42.545 0)
+  (label "CKE_0" (at 73.025 42.545 0)
     (effects (font (size 1.27 1.27)) (justify left bottom))
   )
@@
     (effects (font (size 1.27 1.27)) (justify left bottom))
   )
-  (label "ODT" (at 219.075 60.96 180)
+  (label "ODT_1" (at 219.075 60.96 180)
     (effects (font (size 1.27 1.27)) (justify right bottom))
   )
@@
     (effects (font (size 1.27 1.27)) (justify right bottom))
   )
-  (label "ODT" (at 219.075 136.525 180)
+  (label "ODT_1" (at 219.075 136.525 180)
     (effects (font (size 1.27 1.27)) (justify right bottom))
   )
@@
     (effects (font (size 1.27 1.27)) (justify right bottom))
   )
-  (label "~{CS}" (at 73.025 127 0)
+  (label "~{CS_0}" (at 73.025 127 0)
     (effects (font (size 1.27 1.27)) (justify left bottom))
   )
@@
     (effects (font (size 1.27 1.27)) (justify left bottom))
   )
-  (label "~{DQS}" (at 73.025 76.2 0)
+  (label "~{LDQS}" (at 73.025 76.2 0)
     (effects (font (size 1.27 1.27)) (justify left bottom))
   )
@@
     (effects (font (size 1.27 1.27)) (justify right bottom))
   )
-  (label "~{CS}" (at 219.075 127 180)
+  (label "~{CS_1}" (at 219.075 127 180)
     (effects (font (size 1.27 1.27)) (justify right bottom))
   )
@@
     (effects (font (size 1.27 1.27)) (justify right bottom))
   )
-  (label "ODT" (at 73.025 136.525 0)
+  (label "ODT_0" (at 73.025 136.525 0)
     (effects (font (size 1.27 1.27)) (justify left bottom))
   )
@@
     (effects (font (size 1.27 1.27)) (justify left bottom))
   )
-  (label "DQS" (at 73.025 73.66 0)
+  (label "LDQS" (at 73.025 73.66 0)
     (effects (font (size 1.27 1.27)) (justify left bottom))
   )
@@
     (effects (font (size 1.27 1.27)) (justify left bottom))
   )
-  (label "~{DQS}" (at 73.025 151.765 0)
+  (label "~{UDQS}" (at 73.025 151.765 0)
     (effects (font (size 1.27 1.27)) (justify left bottom))
   )
@@
     (effects (font (size 1.27 1.27)) (justify right bottom))
   )
-  (label "~{CS}" (at 73.025 51.435 0)
+  (label "~{CS_0}" (at 73.025 51.435 0)
     (effects (font (size 1.27 1.27)) (justify left bottom))
   )
@@
     (effects (font (size 1.27 1.27)) (justify left bottom))
   )
-  (label "CKE" (at 219.075 118.11 180)
-    (effects (font (size 1.27 1.27)) (justify right bottom))
-  )
+  (label "CKE_1" (at 219.075 118.11 180)
+    (effects (font (size 1.27 1.27)) (justify right bottom))
+  )
